Commit message: fix xacro files

File: src/lss_arm_description/urdf/lss_arm_5dof.urdf (robot description, URDF)
Before this commit: robot lss_arm_5dof, 10 links, 9 joints
Joints:
- joint lss_arm_joint_7: mimic (none) -> joint=lss_arm_joint_5 multiplier=-1.0 offset=0.0

File: src/lss_arm_description/urdf/lss_gripper_5dof.xacro (robot description, xacro)
@@ -163,5 +163,5 @@
     mesh_offset_rpy="${link_finger_1_mesh_offset}"
     />
-    <!-- mimic_joint="${prefix}${joint_finger_1_name}" -->
+    <!-- mimic_joint="none" -->
     <!-- Finger 2 -->
     <xacro:lss_arm_joint_
@@ -179,5 +179,5 @@
     joint_damping="${joint_finger_2_damping}"
     joint_friction="${joint_finger_2_friction}"
-    mimic_joint="none"
+    mimic_joint="${prefix}${joint_finger_1_name}"
     multiplier="-1.0"
     offset="0.0"
